Commit message: Refactor URDF for 3DOF arm configuration
Updated robot name and joint descriptions to reflect changes in configuration and functionality. Adjusted link dimensions and orientations for better accuracy.

File: urdf/arm_3dof.urdf (robot description, URDF)
Before this commit: robot planar_3dof_arm, 4 links, 3 joints
Joints:
- joint joint2: axis 0 0 1 -> 0 1 0; limit lower=-3.14 upper=3.14 effort=100 velocity=3.0 -> lower=-1.57 upper=1.57 effort=100 velocity=3.0; origin xyz=0.15 0 0 rpy=0 0 0 -> xyz=0 0 0.15 rpy=0 0 0
- joint joint3: axis 0 0 1 -> 0 1 0; limit lower=-3.14 upper=3.14 effort=100 velocity=3.0 -> lower=-2.57 upper=2.57 effort=100 velocity=3.0
